File: atmega32u4-prototyping-board.kicad_pcb (KiCad board)
At the start: 2 copper layers, 40.8 x 25.6 mm, 18 parts, among them J1 USB_C_Receptacle_USB2.0_16P, J2 Conn_01x16, J3 Conn_01x16, U1 ATmega32U4-M, Y1 CSTNE16M0V53C000R0

Commit message: Update board image
Connections:
- R4 pad 1: D- -> D+
- R5 pad 1: D+ -> D-
Routing:
- net D+: track 11.9 -> 10.5 mm
- net D-: track 12.1 -> 11.8 mm, vias 2 -> 0
- added copper zone on F.Cu, net D-
Other:
- board text added: "ATmega32U4 _{Rev 1}"
- board text removed: "ATmega32U4 _{Rev 0}"
Changed lines of the file:
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@@
 		(property ki_fp_filters "C_*")
 		(sheetname "/")
-		(sheetfile "proto.kicad_sch")
+		(sheetfile "atmega32u4-prototyping-board.kicad_sch")
 		(attr smd)
 		(fp_line
@@
 		(property ki_fp_filters "R_*")
 		(sheetname "/")
-		(sheetfile "proto.kicad_sch")
+		(sheetfile "atmega32u4-prototyping-board.kicad_sch")
 		(attr smd)
 		(fp_line
@@
 		(property ki_fp_filters "C_*")
 		(sheetname "/")
-		(sheetfile "proto.kicad_sch")
+		(sheetfile "atmega32u4-prototyping-board.kicad_sch")
 		(attr smd)
 		(fp_line
@@
 		(property ki_fp_filters "R_*")
 		(sheetname "/")
-		(sheetfile "proto.kicad_sch")
+		(sheetfile "atmega32u4-prototyping-board.kicad_sch")
 		(attr smd)
 		(fp_line
@@
 			(layers "F.Cu" "F.Mask" "F.Paste")
 			(roundrect_rratio 0.25)
-			(net 6 "D-")
+			(net 7 "D+")
 			(pintype "passive")
 		)
@@
 		(property ki_fp_filters "C_*")
 		(sheetname "/")
-		(sheetfile "proto.kicad_sch")
+		(sheetfile "atmega32u4-prototyping-board.kicad_sch")
 		(attr smd)
 		(fp_line
@@
 		(property ki_fp_filters "R_*")
 		(sheetname "/")
-		(sheetfile "proto.kicad_sch")
+		(sheetfile "atmega32u4-prototyping-board.kicad_sch")
 		(attr smd)
 		(fp_line
@@
 		(property ki_fp_filters "R_*")
 		(sheetname "/")
-		(sheetfile "proto.kicad_sch")
+		(sheetfile "atmega32u4-prototyping-board.kicad_sch")
 		(attr smd)
 		(fp_line
@@
 		(property ki_fp_filters "C_*")
 		(sheetname "/")
-		(sheetfile "proto.kicad_sch")
+		(sheetfile "atmega32u4-prototyping-board.kicad_sch")
 		(attr smd)
 		(fp_line
@@
 		(property ki_fp_filters "C_*")
 		(sheetname "/")
-		(sheetfile "proto.kicad_sch")
+		(sheetfile "atmega32u4-prototyping-board.kicad_sch")
 		(attr smd)
 		(fp_line
@@
 		(property ki_fp_filters "C_*")
 		(sheetname "/")
-		(sheetfile "proto.kicad_sch")
+		(sheetfile "atmega32u4-prototyping-board.kicad_sch")
 		(attr smd)
 		(fp_line
@@
 		(property ki_fp_filters "C_*")
 		(sheetname "/")
-		(sheetfile "proto.kicad_sch")
+		(sheetfile "atmega32u4-prototyping-board.kicad_sch")
 		(attr smd)
 		(fp_line
@@
 		(property ki_fp_filters "USB*C*Receptacle*")
 		(sheetname "/")
-		(sheetfile "proto.kicad_sch")
+		(sheetfile "atmega32u4-prototyping-board.kicad_sch")
 		(attr smd)
 		(fp_line
@@
 		)
 		(sheetname "/")
-		(sheetfile "proto.kicad_sch")
+		(sheetfile "atmega32u4-prototyping-board.kicad_sch")
 		(attr smd)
 		(fp_line
@@
 		(property ki_fp_filters "R_*")
 		(sheetname "/")
-		(sheetfile "proto.kicad_sch")
+		(sheetfile "atmega32u4-prototyping-board.kicad_sch")
 		(attr smd)
 		(fp_line
@@
 			(layers "F.Cu" "F.Mask" "F.Paste")
 			(roundrect_rratio 0.25)
-			(net 7 "D+")
+			(net 6 "D-")
 			(pintype "passive")
 		)
@@
 		(property ki_fp_filters "QFN*1EP*7x7mm*P0.5mm*")
 		(sheetname "/")
-		(sheetfile "proto.kicad_sch")
+		(sheetfile "atmega32u4-prototyping-board.kicad_sch")
 		(attr smd)
 		(fp_line
@@
 		(property ki_fp_filters "R_*")
 		(sheetname "/")
-		(sheetfile "proto.kicad_sch")
+		(sheetfile "atmega32u4-prototyping-board.kicad_sch")
 		(attr smd)
 		(fp_line
@@
 		(property ki_fp_filters "Connector*:*_1x??_*")
 		(sheetname "/")
-		(sheetfile "proto.kicad_sch")
+		(sheetfile "atmega32u4-prototyping-board.kicad_sch")
 		(attr through_hole)
 		(fp_line
@@
 		(property ki_fp_filters "Connector*:*_1x??_*")
 		(sheetname "/")
-		(sheetfile "proto.kicad_sch")
+		(sheetfile "atmega32u4-prototyping-board.kicad_sch")
 		(attr through_hole)
 		(fp_line
@@
 		)
 	)
-	(gr_text "ATmega32U4\n        _{Rev 0}"
+	(gr_text "ATmega32U4\n        _{Rev 1}"
 		(at 119.698 100.398 0)
 		(layer "F.SilkS")
@@
 	)
 	(segment
-		(start 102.687529 99.648)
-		(end 101.203 99.648)
+		(start 101.203 100.648)
+		(end 100.226 100.648)
 		(width 0.2)
 		(layer "F.Cu")
@@
 	)
 	(segment
-		(start 103.81284 101.262258)
-		(end 102.804561 101.262258)
-		(width 0.7)
+		(start 101.203 99.648)
+		(end 102.600654 99.648)
+		(width 0.2)
 		(layer "F.Cu")
 		(net 6)
 	)
 	(segment
-		(start 102.790547 99.544982)
-		(end 102.687529 99.648)
+		(start 100.226 99.648)
+		(end 101.203 99.648)
 		(width 0.2)
 		(layer "F.Cu")
@@
 	)
 	(segment
-		(start 105.461598 99.6135)
-		(end 103.81284 101.262258)
+		(start 109.539 98.6825)
+		(end 105.118392 98.6825)
 		(width 0.7)
 		(layer "F.Cu")
@@
 	)
 	(segment
-		(start 109.539 99.6135)
-		(end 105.461598 99.6135)
-		(width 0.7)
+		(start 100.177 100.599)
+		(end 100.177 99.697)
+		(width 0.2)
 		(layer "F.Cu")
 		(net 6)
 	)
 	(segment
-		(start 102.804561 101.262258)
-		(end 102.479 100.936697)
-		(width 0.7)
+		(start 102.600654 99.648)
+		(end 102.680154 99.7275)
+		(width 0.2)
 		(layer "F.Cu")
 		(net 6)
 	)
 	(segment
-		(start 101.203 100.648)
-		(end 102.261013 100.648)
-		(width 0.2)
+		(start 104.073392 99.7275)
+		(end 102.680154 99.7275)
+		(width 0.7)
 		(layer "F.Cu")
 		(net 6)
 	)
 	(segment
-		(start 102.261013 100.648)
-		(end 102.361013 100.748)
-		(width 0.2)
+		(start 105.118392 98.6825)
+		(end 104.073392 99.7275)
+		(width 0.7)
 		(layer "F.Cu")
 		(net 6)
 	)
-	(via
-		(at 102.790547 99.544982)
-		(size 0.6)
-		(drill 0.3)
-		(layers "F.Cu" "B.Cu")
-		(net 6)
-	)
-	(via
-		(at 102.361013 100.748)
-		(size 0.6)
-		(drill 0.3)
-		(layers "F.Cu" "B.Cu")
-		(net 6)
-	)
 	(segment
-		(start 102.361013 99.974516)
-		(end 102.790547 99.544982)
+		(start 100.177 99.697)
+		(end 100.226 99.648)
 		(width 0.2)
-		(layer "B.Cu")
+		(layer "F.Cu")
 		(net 6)
 	)
 	(segment
-		(start 102.361013 100.748)
-		(end 102.361013 99.974516)
+		(start 100.226 100.648)
+		(end 100.177 100.599)
 		(width 0.2)
-		(layer "B.Cu")
+		(layer "F.Cu")
 		(net 6)
 	)
 	(segment
-		(start 100.226 100.148)
-		(end 100.177 100.197)
-		(width 0.2)
+		(start 105.461598 99.6135)
+		(end 104.446598 100.6285)
+		(width 0.7)
 		(layer "F.Cu")
 		(net 7)
 	)
 	(segment
-		(start 100.226 101.148)
-		(end 101.203 101.148)
+		(start 102.229 100.197)
+		(end 102.229 101.099)
 		(width 0.2)
 		(layer "F.Cu")
@@
 	)
 	(segment
-		(start 101.203 100.148)
-		(end 100.226 100.148)
+		(start 102.18 101.148)
+		(end 101.203 101.148)
 		(width 0.2)
 		(layer "F.Cu")
@@
 	)
 	(segment
-		(start 109.539 98.6825)
-		(end 105.118392 98.6825)
-		(width 0.7)
-		(layer "F.Cu")
-		(net 7)
-	)
-	(segment
 		(start 101.203 100.148)
-		(end 102.823088 100.148)
+		(end 102.18 100.148)
 		(width 0.2)
 		(layer "F.Cu")
@@
 	)
 	(segment
-		(start 100.177 100.197)
-		(end 100.177 101.099)
-		(width 0.2)
+		(start 109.539 99.6135)
+		(end 105.461598 99.6135)
+		(width 0.7)
 		(layer "F.Cu")
 		(net 7)
 	)
 	(segment
-		(start 105.118392 98.6825)
-		(end 103.439634 100.361258)
+		(start 104.446598 100.6285)
+		(end 102.479 100.6285)
 		(width 0.7)
 		(layer "F.Cu")
@@
 	)
 	(segment
-		(start 100.177 101.099)
-		(end 100.226 101.148)
+		(start 102.229 101.099)
+		(end 102.18 101.148)
 		(width 0.2)
 		(layer "F.Cu")
@@
 	)
 	(segment
-		(start 102.823088 100.148)
-		(end 102.97107 100.295982)
+		(start 102.18 100.148)
+		(end 102.229 100.197)
 		(width 0.2)
 		(layer "F.Cu")
@@
 	)
 	(segment
-		(start 103.439634 100.361258)
-		(end 103.177767 100.361258)
-		(width 0.7)
-		(layer "F.Cu")
-		(net 7)
-	)
-	(segment
 		(start 102.339 99.148)
 		(end 102.839 98.648)
@@
 	)
 	(zone
+		(net 6)
+		(net_name "D-")
+		(layer "F.Cu")
+		(hatch edge 0.5)
+		(priority 1)
+		(connect_pads yes
+			(clearance 0.2)
+		)
+		(min_thickness 0.2)
+		(filled_areas_thickness no)
+		(fill yes
+			(thermal_gap 0.5)
+			(thermal_bridge_width 0.5)
+		)
+		(polygon
+			(pts
+				(xy 103.148 99.377) (xy 101.729 99.377) (xy 101.729 100.079) (xy 103.148 100.079)
+			)
+		)
+	)
+	(zone
 		(net 7)
 		(net_name "D+")
 		(layer "F.Cu")
 		(hatch edge 0.5)
-		(priority 1)
-		(connect_pads
+		(priority 2)
+		(connect_pads yes
 			(clearance 0.2)
 		)
@@
 		(filled_areas_thickness no)
 		(fill yes
-			(thermal_gap 0.2)
-			(thermal_bridge_width 0.2)
+			(thermal_gap 0.5)
+			(thermal_bridge_width 0.5)
 		)
 		(polygon
 			(pts
-				(xy 102.191 100.048) (xy 103.29 100.048) (xy 103.29 100.711) (xy 102.757 100.711) (xy 102.191 100.145)
+				(xy 102.58 100.278) (xy 102.225 100.278) (xy 102.225 100.979) (xy 102.58 100.979)
 			)
 		)
